File: Mini_drone_PCB/Mini_drone_PCB.kicad_pcb (KiCad board)
At the start: 2 copper layers, 30 x 30 mm, 40 parts, among them J1 Power IN, Q1 SS8050, Q2 SS8050, Q3 AO3400, U1 TPS62085RLTR, U2 470nH 6.9mΩ, U3 ESP32-S3-MINI-1, U4 MPU-6050, U5 CH343P, U6 INA236AIDDFR

Commit message: Little fix and add documents
Parts:
- added C13: 0.1uF, Capacitor_SMD:C_0402_1005Metric, F.Cu at (58.3, 70.6)
- added D4: SS34, Diode_SMD:D_SMA, F.Cu at (60.9, 51.0)
- added D5: SS34, Diode_SMD:D_SMA, F.Cu at (60.9, 55.5)
- added D6: SS34, Diode_SMD:D_SMA, F.Cu at (60.9, 60.1)
- added Q4: AO3400, mini_drone:SOT-23-3_L2.9-W1.3-P1.90-LS2.4-BR, F.Cu at (67.1, 50.8)
- added Q5: AO3400, mini_drone:SOT-23-3_L2.9-W1.3-P1.90-LS2.4-BR, F.Cu at (67.1, 55.0)
- added Q6: AO3400, mini_drone:SOT-23-3_L2.9-W1.3-P1.90-LS2.4-BR, F.Cu at (67.1, 59.2)
- added R15: 10k, Capacitor_SMD:C_0402_1005Metric, F.Cu at (70.6, 49.7)
- added R16: 10k, Capacitor_SMD:C_0402_1005Metric, F.Cu at (70.6, 51.7)
- added R17: 10k, Capacitor_SMD:C_0402_1005Metric, F.Cu at (70.6, 53.6)
- added SW1: SW_Push, Button_Switch_SMD:SW_Tactile_SPST_NO_Straight_CK_PTS636Sx25SMTRLFS, F.Cu at (62.1, 67.0)
- moved D3 69.3 mm to (62.0, 39.0)
- moved Q3 69.3 mm to (60.1, 43.4)
- moved R14 69.3 mm to (63.6, 42.3)
- moved C1 48.3 mm to (163.2, 70.8)
- moved C2 48.3 mm to (170.2, 74.8)
- moved R1 48.3 mm to (157.2, 68.8)
- moved R2 48.3 mm to (160.2, 69.8)
- moved R3 48.3 mm to (158.2, 73.8)
- moved U2 48.3 mm to (169.2, 70.8)
- moved U1 48.3 mm to (164.6, 69.2)
- moved U5 48.3 mm to (162.8, 65.5)
- moved USB1 43.2 mm to (113.0, 86.0)
- moved R6 35.9 mm to (115.5, 81.5)
- moved R7 32.4 mm to (110.5, 81.5), turned to 180 degrees
- moved J1 15.6 mm to (126.0, 87.5)
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Connections:
- Q3 pad 1: /Motor Driver/Motor1_PWM -> /MCU/Motor1_PWM
- R14 pad 2: /Motor Driver/Motor1_PWM -> /MCU/Motor1_PWM
- U3 pad 10: unconnected-(U3-IO6-Pad10) -> /MCU/Motor3_PWM
- U3 pad 11: unconnected-(U3-IO7-Pad11) -> /MCU/Motor4_PWM
- U3 pad 8: unconnected-(U3-IO4-Pad8) -> /MCU/Motor1_PWM
- U3 pad 9: unconnected-(U3-IO5-Pad9) -> /MCU/Motor2_PWM
- U6 pad 5: /PSU/INA236_SCL -> /MCU/ESP_SCL
- U6 pad 6: /PSU/INA236_SDA -> /MCU/ESP_SDA
Routing:
- net GND: track 0.00 -> 4.44 mm
- net Net-(USB1-CC1): track 0.00 -> 2.44 mm
- net Net-(USB1-CC2): track 0.00 -> 2.24 mm
Other:
- board size 30 x 30 mm -> 6.5 x 0.7 mm

Commit message: more info
Connections:
- Q2 pad 2: /MCU/GPIO0 -> /MCU/DTR
- Q2 pad 3: /MCU/DTR -> /MCU/GPIO0
Changed lines of the file:
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@@
 			(layers "F.Cu" "F.Mask" "F.Paste")
 			(roundrect_rratio 0.25)
-			(net 37 "/MCU/GPIO0")
+			(net 40 "/MCU/DTR")
 			(pinfunction "E")
 			(pintype "passive")
@@
 			(layers "F.Cu" "F.Mask" "F.Paste")
 			(roundrect_rratio 0.25)
-			(net 40 "/MCU/DTR")
+			(net 37 "/MCU/GPIO0")
 			(pinfunction "C")
 			(pintype "passive")
