File: Mini_drone_PCB/_autosave-Mini_drone_PCB.kicad_pcb (KiCad board)
At the start: 2 copper layers, 45.7 x 42.9 mm, 56 parts, among them J1 XT30PW-M, Q1 SS8050, Q2 SS8050, Q3 AO3400, Q4 AO3400, Q5 AO3400, Q6 AO3400, Q7 AO4407A, SW1 SW_Push, SW2 Slide_switch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

Commit message: fix sch
Routing:
- net /MCU/ESP_SDA: track 8.13 -> 76.9 mm, vias 0 -> 2
- net /MCU/ESP_SCL: track 8.07 -> 68.2 mm, vias 0 -> 2
