File: Mini_drone_PCB/Mini_drone_PCB.kicad_sch (KiCad schematic)
At the start: 0 parts

Commit message: Little fix and add documents
Changed lines of the file:
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@@
-	)
-	(junction
-		(at 115.57 102.87)
-		(diameter 0)
-		(color 0 0 0 0)
 	)
 	(junction
@@
 		(diameter 0)
 		(color 0 0 0 0)
-	)
-	(junction
-		(at 119.38 105.41)
-		(diameter 0)
-		(color 0 0 0 0)
-	)
-	(wire
-		(pts
-			(xy 115.57 123.19) (xy 115.57 102.87)
-		)
-		(stroke
-			(width 0)
-			(type default)
-		)
 	)
 	(wire
@@
 	(wire
 		(pts
-			(xy 106.68 105.41) (xy 119.38 105.41)
-		)
-		(stroke
-			(width 0)
-			(type default)
-		)
-	)
-	(wire
-		(pts
 			(xy 119.38 95.25) (xy 119.38 100.33)
 		)
@@
 	(wire
 		(pts
-			(xy 115.57 102.87) (xy 115.57 97.79)
+			(xy 115.57 97.79) (xy 115.57 123.19)
 		)
 		(stroke
@@
 	(wire
 		(pts
-			(xy 119.38 100.33) (xy 119.38 105.41)
-		)
-		(stroke
-			(width 0)
-			(type default)
-		)
-	)
-	(wire
-		(pts
-			(xy 106.68 102.87) (xy 115.57 102.87)
+			(xy 119.38 100.33) (xy 119.38 125.73)
 		)
 		(stroke
@@
 		)
 		(stroke
-			(width 0)
-			(type default)
-		)
-	)
-	(wire
-		(pts
-			(xy 119.38 125.73) (xy 119.38 105.41)
-		)
-		(stroke

Commit message: Route_Finished
Parts:
- added H1, H2, H3, H4: MountingHole_Pad, MountingHole:MountingHole_2.5mm_Pad, symbol Mechanical:MountingHole_Pad
Connections:
- no-connect marks 0 -> 4
