File: Mini_drone_PCB/MCU.kicad_sch (KiCad schematic)
At the start: 19 parts, among them Q1 SS8050, Q2 SS8050, SW1 SW_Push, U3 ESP32-S3-MINI-1, U5 CH343P

Commit message: Little fix and add documents
Connections:
- net DTR: now also Q2.2 (E); no longer Q2.3 (C)
- net GPIO0: now also Q2.3 (C); no longer Q2.2 (E)
Other:
- note added: "Ref:documents/AI-S3 ESP32-S3 Dev Board Schematic.pdf"

Commit message: fix sch
Parts:
- added C14: 0.1uF, Capacitor_SMD:C_0402_1005Metric, symbol Device:C
- added U7: USBLC6-2P6, Package_TO_SOT_SMD:SOT-666, symbol Power_Protection:USBLC6-2P6
Connections:
- net D+: now also U7.4 (I/O2); no longer USB1.6 (DP1), USB1.8 (DP2)
- net D-: now also U7.6 (I/O1); no longer USB1.5 (DN2), USB1.7 (DN1)
- net GND: now also C14.2, U7.2 (GND)
- net +BATT renamed +VBUS
- net +VBUS: now also C14.1, U7.5 (VBUS)
- new net: U7.1 (I/O1), USB1.5 (DN2), USB1.7 (DN1)
- new net: U7.3 (I/O2), USB1.6 (DP1), USB1.8 (DP2)
Other:
- moved on the sheet: C7, C8, Q1, Q2, R10, R11, R6, R7, U5

Commit message: Route_Finished
Parts:
- C11: LCSC Part # C59461 -> C15525
- C9: LCSC Part # C59461 -> C14445
- R10, R11, R12: LCSC Part # C25531 -> C25531
- U3: LCSC Part # C2913206 -> C2913206
- U5: LCSC Part # C2846043 -> C2846043
Changed lines of the file:
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@@
 			)
 		)
-		(property "LCSC Part #" " C25531"
+		(property "LCSC Part #" "C25531"
 			(at 218.44 27.94 90)
 			(effects
@@
 			)
 		)
-		(property "LCSC Part #" "C59461"
+		(property "LCSC Part #" "C15525"
 			(at 193.04 33.02 0)
 			(effects
@@
 			)
 		)
-		(property "LCSC Part #" " C2913206 "
+		(property "LCSC Part #" "C2913206 "
 			(at 236.22 78.74 0)
 			(effects
@@
 			)
 		)
-		(property "LCSC Part #" "C59461"
+		(property "LCSC Part #" "C14445 "
 			(at 218.44 38.1 0)
 			(effects
@@
 			)
 		)
-		(property "LCSC Part #" " C25531"
+		(property "LCSC Part #" "C25531"
 			(at 97.79 118.11 90)
 			(effects
@@
 			)
 		)
-		(property "LCSC Part #" " C2846043"
+		(property "LCSC Part #" "C2846043"
 			(at 43.18 128.27 0)
 			(effects
@@
 			)
 		)
-		(property "LCSC Part #" " C25531"
+		(property "LCSC Part #" "C25531"
 			(at 97.79 135.89 90)
 			(effects

Commit message: Verified and Finished
Other:
- note added: "Checked"
Changed lines of the file:
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@@
+		)
+	)
+	(text "Checked"
+		(exclude_from_sim no)
+		(at 36.576 68.834 0)
+		(effects
+			(font
+				(face "KiCad Font")
+				(size 1.27 1.27)
+				(thickness 0.254)
+				(bold yes)
+				(color 255 63 23 1)
+			)
 		)
 	)
@@
 		)
 	)
+	(text "Checked"
+		(exclude_from_sim no)
+		(at 174.752 45.72 0)
+		(effects
+			(font
+				(face "KiCad Font")
+				(size 1.27 1.27)
+				(thickness 0.254)
+				(bold yes)
+				(color 255 63 23 1)
+			)
+		)
+	)
+	(text "Checked"
+		(exclude_from_sim no)
+		(at 114.554 127 0)
+		(effects
+			(font
+				(face "KiCad Font")
+				(size 1.27 1.27)
+				(thickness 0.254)
+				(bold yes)
+				(color 255 63 23 1)
+			)
+		)
+	)
+	(text "Checked"
+		(exclude_from_sim no)
+		(at 214.122 66.548 0)
+		(effects
+			(font
+				(face "KiCad Font")
+				(size 1.27 1.27)
+				(thickness 0.254)
+				(bold yes)
+				(color 255 63 23 1)
+			)
+		)
+	)
 	(text "Ref:documents/AI-S3 ESP32-S3 Dev Board Schematic.pdf"
 		(exclude_from_sim no)
@@
 			(font
 				(size 1.27 1.27)
+			)
+		)
+	)
+	(text "Checked"
+		(exclude_from_sim no)
+		(at 245.11 108.966 0)
+		(effects
+			(font
+				(face "KiCad Font")
+				(size 1.27 1.27)
+				(thickness 0.254)
+				(bold yes)
+				(color 255 63 23 1)
+			)
+		)
+	)
+	(text "Checked"
+		(exclude_from_sim no)
+		(at 89.916 46.99 0)
+		(effects
+			(font
+				(face "KiCad Font")
+				(size 1.27 1.27)
+				(thickness 0.254)
+				(bold yes)
+				(color 255 63 23 1)
 			)
 		)
@@
 			)
 		)
+	)
+	(text "Checked"
+		(exclude_from_sim no)
+		(at 58.42 146.304 0)
+		(effects
+			(font
+				(face "KiCad Font")
+				(size 1.27 1.27)
+				(thickness 0.254)
+				(bold yes)
+				(color 255 63 23 1)
+			)
+		)
+	)
+	(text "Checked"
+		(exclude_from_sim no)
+		(at 214.63 43.942 0)
+		(effects
+			(font
+				(face "KiCad Font")
+				(size 1.27 1.27)
+				(thickness 0.254)
+				(bold yes)
+				(color 255 63 23 1)
+			)
+		)
+	)
+	(text "Checked"
+		(exclude_from_sim no)
+		(at 214.884 93.726 0)
+		(effects
+			(font
+				(face "KiCad Font")
+				(size 1.27 1.27)
+				(thickness 0.254)
+				(bold yes)
+				(color 255 63 23 1)
+			)
+		)
+	)
+	(text "Checked"
+		(exclude_from_sim no)
+		(at 196.342 77.47 0)
+		(effects
+			(font
+				(face "KiCad Font")
+				(size 1.27 1.27)
+				(thickness 0.254)
+				(bold yes)
+				(color 255 63 23 1)
+			)
+		)
