File: Mini_drone_PCB/PSU.kicad_sch (KiCad schematic)
At the start: 15 parts, among them J1 Power IN, U1 TPS62085RLTR, U2 470nH 6.9mΩ, U6 INA236AIDDFR

Commit message: Little fix and add documents
Other:
- note added: "Ref:https://item.szlcsc.com/datasheet/INA236AIDDFR/6333219.html"

Commit message: fix sch
Parts:
- removed J1: Power IN, Connector_JST:JST_PH_S2B-PH-K_1x02_P2.00mm_Horizontal, symbol Connector:Conn_01x02_Pin
- added D7, D8: PMEG2010ER, Diode_SMD:Nexperia_CFP3_SOD-123W, symbol Diode:PMEG2010ER
- added J1: XT30PW-M, Sharing_Footprint:AMASS_XT30PW-M, symbol Sharing_Symbol:XT30PW-M
- added SW2: Slide_switch, mini_drone:SW-SMD_SSSS811101, symbol mini_drone:SSSS811101
Connections:
- net +BATT: no longer C1.1, R13.1, U1.7 (VIN), U6.2 (IN-)
- net GND: now also J1.1 (-)
- net at R13.2, U6.1 (IN+): now also J1.2 (+)
- new net: C1.1, D7.1 (K), D8.1 (K), U1.7 (VIN)
- new net: D8.2 (A), SW2.2
- new net +VBUS: D7.2 (A)
- new net +VIN: R13.1, SW2.1, U6.2 (IN-)
- no-connect marks 1 -> 5
Other:
- moved on the sheet: C1, C12, C2, D1, D2, R1, R13, R2, R3, R8, R9, U1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

Commit message: update_sch_and_PCB
Parts:
- removed D1: VBAT LED, LED_SMD:LED_0603_1608Metric, symbol Device:LED
- removed R8: 510, Capacitor_SMD:C_0402_1005Metric, symbol Device:R
Connections:
- net +BATT: now also R13.1, SW2.1, U6.2 (IN-); no longer U1.1 (EN)
- net +VIN: now also C1.1, D7.1 (K), D8.1 (K), U1.1 (EN), U1.7 (VIN); no longer R13.1, SW2.1, U6.2 (IN-)
Other:
- note added: "Current sense"
- note added: "ORing diode"
- moved on the sheet: D2, R9

Commit message: Route_Finished
Parts:
- added D1, D9: LED, LED_THT:LED_D3.0mm_Horizontal_O6.35mm_Z2.0mm, symbol Device:LED
- added R18, R8: 510, Capacitor_SMD:C_0402_1005Metric, symbol Device:R
- C1: LCSC Part # C1691 -> C15525
- R1: LCSC Part # C23192 -> C11616
- R13: LCSC Part # C2846043 -> C105366
- R2: LCSC Part # C22815 -> C185462
- R3: LCSC Part # C22935 -> C26083
- R9: value 220 -> 510; LCSC Part # C2909336 -> C25123
- SW2: LCSC Part # (none) -> C109335
Connections:
- net +3V3: now also R18.1, R8.1
- net GND: now also D1.1 (K), D9.1 (K)
- new net: D9.2 (A), R18.2
- new net: D1.2 (A), R8.2
Other:
- moved on the sheet: D2, R9

Commit message: Verified and Finished
Parts:
- added C15: 220uF, Capacitor_SMD:CP_Elec_6.3x5.4, symbol Device:C_Polarized
- C2: LCSC Part # C59461 -> C105226
- D1, D9: LCSC Part # C86881 -> (none)
Connections:
- net GND: now also C15.2
- net at J1.2 (+), R13.2, U6.1 (IN+): now also C15.1
Other:
- note added: "Checked"
- moved on the sheet: J1
