File: Mini_drone_PCB/sensor.kicad_sch (KiCad schematic)
At the start: 7 parts, among them J2 VL53L1X ToF Pogo, J3 PMW3901 Optical Flow Pogo, U4 MPU-6050

Commit message: Little fix and add documents
Other:
- note added: "https://invensense.tdk.com/wp-content/uploads/2015/02/MPU-6000-Datasheet1.pdf"
Changed lines of the file:
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@@
+		)
+	)
+	(text "https://invensense.tdk.com/wp-content/uploads/2015/02/MPU-6000-Datasheet1.pdf"
+		(exclude_from_sim no)
+		(at 212.852 81.28 0)
+		(effects
+			(font
+				(size 1.27 1.27)
+			)
 		)
 	)

Commit message: Route_Finished
Parts:
- C3: LCSC Part # C1691 -> C15195
- C6: LCSC Part # C1691 -> C1531
- J2: footprint (none) -> mini_drone:POGO 4Pin Pitch 2.54
- J3: footprint (none) -> mini_drone:POGO 6Pin Pitch 2.54
Connections:
- net GND: now also J2.4 (Pin_4), J3.6 (Pin_6); no longer J2.2 (Pin_2), J3.2 (Pin_2)
- net PWM3901_CS: now also J3.5 (Pin_5); no longer J3.6 (Pin_6)
- net PWM3901_MISO: now also J3.4 (Pin_4); no longer J3.5 (Pin_5)
- net PWM3901_MOSI: now also J3.2 (Pin_2); no longer J3.3 (Pin_3)
- net PWM3901_SCLK: now also J3.3 (Pin_3); no longer J3.4 (Pin_4)
- net VL53L1X_SCL: now also J2.3 (Pin_3); no longer J2.4 (Pin_4)
- net VL53L1X_SDA: now also J2.2 (Pin_2); no longer J2.3 (Pin_3)
Changed lines of the file:
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@@
 	(wire
 		(pts
-			(xy 31.75 113.03) (xy 46.99 113.03)
-		)
-		(stroke
-			(width 0)
-			(type default)
-		)
-	)
-	(wire
-		(pts
 			(xy 95.25 29.21) (xy 99.06 29.21)
 		)
@@
 	(wire
 		(pts
-			(xy 78.74 109.22) (xy 93.98 109.22)
-		)
-		(stroke
-			(width 0)
-			(type default)
-		)
-	)
-	(wire
-		(pts
 			(xy 76.2 48.26) (xy 76.2 55.88)
 		)
@@
 		)
 	)
-	(hierarchical_label "PWM3901_MOSI"
-		(shape input)
-		(at 93.98 111.76 180)
+	(hierarchical_label "MPU_SCL"
+		(shape bidirectional)
+		(at 83.82 45.72 180)
 		(effects
 			(font
@@
 		)
 	)
-	(hierarchical_label "PWM3901_CS"
+	(hierarchical_label "PWM3901_SCLK"
 		(shape input)
-		(at 93.98 119.38 180)
+		(at 93.98 111.76 180)
 		(effects
 			(font
@@
 		)
 	)
-	(hierarchical_label "PWM3901_MISO"
-		(shape output)
-		(at 93.98 116.84 180)
+	(hierarchical_label "VL53L1X_SDA"
+		(shape bidirectional)
+		(at 46.99 113.03 180)
 		(effects
 			(font
@@
 		)
 	)
-	(hierarchical_label "MPU_SCL"
-		(shape bidirectional)
-		(at 83.82 45.72 180)
+	(hierarchical_label "PWM3901_CS"
+		(shape input)
+		(at 93.98 116.84 180)
 		(effects
 			(font
@@
 		)
 	)
-	(hierarchical_label "PWM3901_SCLK"
+	(hierarchical_label "PWM3901_MOSI"
 		(shape input)
-		(at 93.98 114.3 180)
+		(at 93.98 109.22 180)
 		(effects
 			(font
@@
 		)
 	)
-	(hierarchical_label "VL53L1X_SDA"
-		(shape bidirectional)
-		(at 46.99 115.57 180)
+	(hierarchical_label "PWM3901_MISO"
+		(shape output)
+		(at 93.98 114.3 180)
 		(effects
 			(font
@@
 	(hierarchical_label "VL53L1X_SCL"
 		(shape bidirectional)
-		(at 46.99 118.11 180)
+		(at 46.99 115.57 180)
 		(effects
 			(font
@@
 	(symbol
 		(lib_id "power:GNDD")
-		(at 31.75 113.03 270)
+		(at 46.99 118.11 270)
 		(unit 1)
 		(exclude_from_sim no)
@@
 		(fields_autoplaced yes)
 		(property "Reference" "#PWR012"
-			(at 25.4 113.03 0)
+			(at 40.64 118.11 0)
 			(effects
 				(font
@@
 		)
 		(property "Value" "GND"
-			(at 27.94 113.0299 90)
+			(at 43.18 118.1099 90)
 			(effects
 				(font
@@
 		)
 		(property "Footprint" ""
-			(at 31.75 113.03 0)
+			(at 46.99 118.11 0)
 			(effects
 				(font
@@
 		)
 		(property "Datasheet" ""
-			(at 31.75 113.03 0)
+			(at 46.99 118.11 0)
 			(effects
 				(font
@@
 		)
 		(property "Description" "Power symbol creates a global label with name \"GNDD\" , digital ground"
-			(at 31.75 113.03 0)
+			(at 46.99 118.11 0)
 			(effects
 				(font
@@
 			)
 		)
-		(property "LCSC Part #" "C1691"
+		(property "LCSC Part #" "C15195 "
 			(at 91.44 29.21 0)
 			(effects
@@
 	(symbol
 		(lib_id "power:GNDD")
-		(at 78.74 109.22 270)
+		(at 93.98 119.38 270)
 		(unit 1)
 		(exclude_from_sim no)
@@
 		(fields_autoplaced yes)
 		(property "Reference" "#PWR014"
-			(at 72.39 109.22 0)
+			(at 87.63 119.38 0)
 			(effects
 				(font
@@
 		)
 		(property "Value" "GND"
-			(at 74.93 109.2199 90)
+			(at 90.17 119.3799 90)
 			(effects
 				(font
@@
 		)
 		(property "Footprint" ""
-			(at 78.74 109.22 0)
+			(at 93.98 119.38 0)
 			(effects
 				(font
@@
 		)
 		(property "Datasheet" ""
-			(at 78.74 109.22 0)
+			(at 93.98 119.38 0)
 			(effects
 				(font
@@
 		)
 		(property "Description" "Power symbol creates a global label with name \"GNDD\" , digital ground"
-			(at 78.74 109.22 0)
+			(at 93.98 119.38 0)
 			(effects
 				(font
@@
 			)
 		)
-		(property "Footprint" ""
+		(property "Footprint" "mini_drone:POGO 6Pin Pitch 2.54"
 			(at 99.06 111.76 0)
 			(effects
@@
 			)
 		)
-		(property "Footprint" ""
+		(property "Footprint" "mini_drone:POGO 4Pin Pitch 2.54"
 			(at 52.07 113.03 0)
 			(effects
@@
 			)
 		)
-		(property "LCSC Part #" "C1691"
+		(property "LCSC Part #" "C1531 "
 			(at 134.62 55.88 0)
 			(effects

Commit message: Verified and Finished
Other:
- note added: "Checked"
Changed lines of the file:
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@@
+		)
+	)
+	(text "Checked"
+		(exclude_from_sim no)
+		(at 50.8 120.904 0)
+		(effects
+			(font
+				(face "KiCad Font")
+				(size 1.27 1.27)
+				(thickness 0.254)
+				(bold yes)
+				(color 255 63 23 1)
+			)
+		)
+	)
+	(text "Checked"
+		(exclude_from_sim no)
+		(at 102.108 121.92 0)
+		(effects
+			(font
+				(face "KiCad Font")
+				(size 1.27 1.27)
+				(thickness 0.254)
+				(bold yes)
+				(color 255 63 23 1)
+			)
+		)
+	)
+	(text "Checked"
+		(exclude_from_sim no)
+		(at 107.696 72.39 0)
+		(effects
+			(font
+				(face "KiCad Font")
+				(size 1.27 1.27)
+				(thickness 0.254)
+				(bold yes)
+				(color 255 63 23 1)
+			)
 		)
 	)
